File: hardware/TetrisEarrings.kicad_sch (KiCad schematic)
At the start: 106 parts, among them J1 TC2030-IDC-NL, J2 DOCK, Q1 AO3401A, Q2 2N7002, SW1 BTN, U1 STM32F070F6P6, U2 MCP73831-2, U3 ME6211C33, Y1 8MHz

Commit message: fixup! Hardware spec
Parts:
- SW1: footprint Button_Switch_SMD:SW_SPST_PTS645 -> Button_Switch_SMD:SW_Push_1P1T_NO_CK_KMR2
Connections:
- net GND: now also Y1.2 (GND), Y1.4 (GND)
- net OSC_OUT: now also Y1.3; no longer Y1.2

Commit message: Add KiCad project files for Tetris Earrings: schematic, PCB, scripts, BOM, CPL, and fab outputs
Parts:
- J1, J2: now left out of the parts list
Connections:
- net OSC_IN: now also Y1.3; no longer Y1.1
- net OSC_OUT: now also Y1.1; no longer Y1.3
Changed lines of the file:
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@@
     (instances (project "TetrisEarrings" (path "/0f8a0f60-1e7e-4a3b-9d2c-7c1e5f4b6a01" (reference "BT1") (unit 1))))
   )
-  (symbol (lib_id "TetrisEarrings:Pads_2") (at 64.77 59.69 0) (unit 1) (exclude_from_sim no) (in_bom yes) (on_board yes) (dnp no)
+  (symbol (lib_id "TetrisEarrings:Pads_2") (at 64.77 59.69 0) (unit 1) (exclude_from_sim no) (in_bom no) (on_board yes) (dnp no)
     (property "Reference" "J2" (at 69.85 58.42 0) (effects (font (size 1.27 1.27))))
     (property "Value" "DOCK" (at 69.85 60.96 0) (effects (font (size 1.27 1.27))))
@@
     (instances (project "TetrisEarrings" (path "/0f8a0f60-1e7e-4a3b-9d2c-7c1e5f4b6a01" (reference "C10") (unit 1))))
   )
-  (symbol (lib_id "TetrisEarrings:TC2030_SWD") (at 199.39 199.39 0) (unit 1) (exclude_from_sim no) (in_bom yes) (on_board yes) (dnp no)
+  (symbol (lib_id "TetrisEarrings:TC2030_SWD") (at 199.39 199.39 0) (unit 1) (exclude_from_sim no) (in_bom no) (on_board yes) (dnp no)
     (property "Reference" "J1" (at 199.39 189.23 0) (effects (font (size 1.27 1.27))))
     (property "Value" "TC2030-IDC-NL" (at 199.39 209.55 0) (effects (font (size 1.27 1.27))))
@@
   (label "BOOT0" (at 180.34 93.98 90) (effects (font (size 1.27 1.27)) (justify left bottom)))
   (label "NRST" (at 199.39 104.14 90) (effects (font (size 1.27 1.27)) (justify left bottom)))
-  (label "OSC_IN" (at 184.15 144.78 180) (effects (font (size 1.27 1.27)) (justify right bottom)))
-  (label "OSC_OUT" (at 196.85 144.78 0) (effects (font (size 1.27 1.27)) (justify left bottom)))
+  (label "OSC_OUT" (at 184.15 144.78 180) (effects (font (size 1.27 1.27)) (justify right bottom)))
+  (label "OSC_IN" (at 196.85 144.78 0) (effects (font (size 1.27 1.27)) (justify left bottom)))
   (label "OSC_IN" (at 175.26 153.67 90) (effects (font (size 1.27 1.27)) (justify left bottom)))
   (label "OSC_OUT" (at 204.47 153.67 90) (effects (font (size 1.27 1.27)) (justify left bottom)))
